File: Hardware/PCB/G431KB_imu_Project.kicad_sch (KiCad schematic)
At the start: 27 parts, among them U1 STM32G431KBUx, U2 BMM350_C17225907, U3 ICM-45686, U4 ICM-45686, U5 TPS7A20xxxDQN, Y1 16Mhz

Commit message: 1.1.0
对硬件进行了修改，去除了5v容忍，更改了ldo以修复bmm350的供电错误问题
Parts:
- added D2: BZX584C3V6, easyeda2kicad:SOD-523_L1.2-W0.8-LS1.6-RD-1, symbol easyeda2kicad:BZX584C3V6
- P1, P2: footprint User_footprints:6Pin半孔 -> User_footprints:6Pin2.54
Connections:
- net GND: now also D2.2 (A)
- net VDD: now also C8.1, U2.B3 (VDDIO), U5.3 (EN), U5.4 (IN), D2.1 (C); no longer C9.1, U2.C1 (VDD), U5.1 (OUT)
- removed net VIN: C14.1, P1.1, U5.3 (EN), U5.4 (IN)
- new net +1.8: C14.1, C9.1, U2.C1 (VDD), U5.1 (OUT)
- no-connect marks 14 -> 15
Changed lines of the file:
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@@
 	)
 	(no_connect
+		(at 260.35 135.89)
+	)
+	(no_connect
 		(at 257.81 91.44)
 	)
@@
 	(wire
 		(pts
+			(xy 238.76 125.73) (xy 245.11 125.73)
+		)
+		(stroke
+			(width 0)
+			(type default)
+		)
+	)
+	(wire
+		(pts
 			(xy 43.18 97.79) (xy 54.61 97.79)
 		)
@@
 	(wire
 		(pts
+			(xy 259.08 125.73) (xy 255.27 125.73)
+		)
+		(stroke
+			(width 0)
+			(type default)
+		)
+	)
+	(wire
+		(pts
 			(xy 91.44 102.87) (xy 80.01 102.87)
 		)
@@
 	(wire
 		(pts
-			(xy 273.05 135.89) (xy 260.35 135.89)
-		)
-		(stroke
-			(width 0)
-			(type default)
-		)
-	)
-	(wire
-		(pts
 			(xy 148.59 96.52) (xy 158.75 96.52)
 		)
@@
 		)
 	)
-	(label "VIN"
+	(label "+1.8"
 		(at 107.95 170.18 270)
 		(effects
@@
 		)
 	)
+	(label "VDD"
+		(at 238.76 125.73 0)
+		(effects
+			(font
+				(size 1.27 1.27)
+			)
+			(justify left bottom)
+		)
+	)
 	(label "SPI1_SCLK"
 		(at 91.44 87.63 180)
@@
 		)
 	)
-	(label "VIN"
+	(label "VDD"
 		(at 111.76 137.16 90)
 		(effects
@@
 		)
 	)
-	(label "VDD"
+	(label "+1.8"
 		(at 160.02 127 0)
 		(effects
@@
 		)
 	)
-	(label "VIN"
-		(at 273.05 135.89 180)
-		(effects
-			(font
-				(size 1.27 1.27)
-				(thickness 0.1588)
-			)
-			(justify right bottom)
-		)
-	)
 	(label "UART1_RX"
 		(at 227.33 146.05 0)
@@
 		)
 	)
-	(label "VIN"
+	(label "VDD"
 		(at 44.45 173.99 0)
 		(effects
@@
 		)
 	)
-	(label "VDD"
+	(label "+1.8"
 		(at 191.77 144.78 180)
 		(effects
@@
 		)
 	)
-	(label "VDD"
+	(label "+1.8"
 		(at 77.47 173.99 180)
 		(effects
@@
 		)
 	)
+	(label "VDD"
+		(at 189.23 147.32 180)
+		(effects
+			(font
+				(size 1.27 1.27)
+			)
+			(justify right bottom)
+		)
+	)
 	(label "IO1"
 		(at 227.33 143.51 0)
@@
 		(on_board yes)
 		(dnp no)
-		(fields_autoplaced yes)
 		(property "Reference" "P2"
-			(at 248.92 141.6049 0)
+			(at 243.586 131.572 0)
 			(effects
 				(font
@@
 			)
 		)
-		(property "Footprint" "User_footprints:6Pin半孔"
+		(property "Footprint" "User_footprints:6Pin2.54"
 			(at 245.11 152.4 0)
 			(effects
@@
 		(on_board yes)
 		(dnp no)
-		(fields_autoplaced yes)
 		(property "Reference" "P1"
-			(at 255.27 129.54 0)
+			(at 255.27 131.318 0)
 			(effects
 				(font
@@
 			)
 		)
-		(property "Footprint" "User_footprints:6Pin半孔"
+		(property "Footprint" "User_footprints:6Pin2.54"
 			(at 255.27 132.08 0)
 			(effects
@@
 	)
 	(symbol
+		(lib_id "easyeda2kicad:BZX584C3V6")
+		(at 250.19 125.73 0)
+		(unit 1)
+		(exclude_from_sim no)
+		(in_bom yes)
+		(on_board yes)
+		(dnp no)
+		(fields_autoplaced yes)
+		(property "Reference" "D2"
+			(at 250.19 119.38 0)
+			(effects
+				(font
+					(size 1.27 1.27)
+				)
+			)
+		)
+		(property "Value" "BZX584C3V6"
+			(at 250.19 121.92 0)
+			(effects
+				(font
+					(size 1.27 1.27)
+				)
+			)
+		)
+		(property "Footprint" "easyeda2kicad:SOD-523_L1.2-W0.8-LS1.6-RD-1"
+			(at 250.19 133.35 0)
+			(effects
+				(font
+					(size 1.27 1.27)
+				)
+				(hide yes)
+			)
+		)
+		(property "Datasheet" ""
+			(at 250.19 125.73 0)
+			(effects
+				(font
+					(size 1.27 1.27)
+				)
+				(hide yes)
+			)
+		)
+		(property "Description" ""
+			(at 250.19 125.73 0)
+			(effects
+				(font
+					(size 1.27 1.27)
+				)
+				(hide yes)
+			)
+		)
+		(property "LCSC Part" "C22395574"
+			(at 250.19 135.89 0)
+			(effects
+				(font
+					(size 1.27 1.27)
+				)
+				(hide yes)
+			)
+		)
+		(pin "1"
+		)
+		(pin "2"
+		)
+		(instances
+			(project ""
+				(path "/5661f608-9224-4e9d-b6ec-46f504ea7c13"
+					(reference "D2")
+					(unit 1)
+				)
+			)
+		)
+	)
+	(symbol
 		(lib_id "Device:C")
 		(at 38.1 127 0)
@@
 					(unit 1)
 				)
+			)
+		)
+	)
+	(symbol
+		(lib_id "power:GND")
+		(at 259.08 125.73 90)
+		(unit 1)
+		(exclude_from_sim no)
+		(in_bom yes)
+		(on_board yes)
+		(dnp no)
+		(fields_autoplaced yes)
+		(property "Reference" "#PWR023"
+			(at 265.43 125.73 0)
+			(effects
+				(font
+					(size 1.27 1.27)
+				)
+				(hide yes)
+			)
+		)
+		(property "Value" "GND"
+			(at 262.89 125.7299 90)
+			(effects
+				(font
+					(size 1.27 1.27)
+				)
+				(justify right)
+			)
+		)
+		(property "Footprint" ""
+			(at 259.08 125.73 0)
+			(effects
+				(font
+					(size 1.27 1.27)
+				)
+				(hide yes)
+			)
+		)
+		(property "Datasheet" ""
+			(at 259.08 125.73 0)
+			(effects
+				(font
+					(size 1.27 1.27)
+				)
+				(hide yes)
+			)
+		)
+		(property "Description" "Power symbol creates a global label with name \"GND\" , ground"
+			(at 259.08 125.73 0)
+			(effects
+				(font
+					(size 1.27 1.27)
+				)
+				(hide yes)
+			)
+		)
+		(pin "1"
+		)
+		(instances
+			(project "G431KB_imu_Project"
+				(path "/5661f608-9224-4e9d-b6ec-46f504ea7c13"
+					(reference "#PWR023")
+					(unit 1)
+				)
